File: EPSM YMF288 Modular Famicom Horizontal/EPSM YMF288 Modular Famicom Horizontal-rounded.kicad_pcb (KiCad board)
At the start: 2 copper layers, 99 x 91.7 mm, 35 parts, among them J1 EPSM_DATA, J2 EPSM_AUDIO, J3 EPSM_SND_OUT, J4 EPSM_ADDR, J5 CONSOLE_M, J6 CARTRIDGE_F, U1 YMF288, U2 74HCT541, U3 74HCT541, U4 74HCT541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

Commit message: Adjust routing
Parts:
- removed the Ref** at (138.4, 87.0)
- added svg2mod: G***, EPSM YMF288 Modular Famicom Horizontal:maustech icon fiducial 0-50mm 1-50mm, F.Cu at (138.4, 87.0)
- moved R1 34.8 mm to (130.2, 47.6), turned to 180 degrees
- moved D1 34.6 mm to (130.2, 49.5), turned to 180 degrees
Routing:
- net VCC: track 86.1 -> 82.8 mm, vias 70 -> 69
- net /B_CPU_A4: track 13.3 -> 12.7 mm
- net /~{IRQ}: track 83.4 -> 82.9 mm
- net /AUD_RF: track 75.9 -> 75.4 mm
- net GND: vias 195 -> 196
