File: EPSM YMF288 Modular Famicom Horizontal/EPSM YMF288 Modular Famicom Horizontal-rounded.kicad_pcb (KiCad board)
At the start: 2 copper layers, 99 x 91.7 mm, 35 parts, among them J1 EPSM_DATA, J2 EPSM_AUDIO, J3 EPSM_SND_OUT, J4 EPSM_ADDR, J5 CONSOLE_M, J6 CARTRIDGE_F, U1 YMF288, U2 74HCT541, U3 74HCT541, U4 74HCT541, U5 74HCT541, X1 SG-8002CA

Commit message: fix: Update processed rounded tracks
Parts:
- added C11: 0.1uF, Capacitor_SMD:C_0805_2012Metric_Pad1.18x1.45mm_HandSolder, F.Cu at (148.6, 71.1)
- added JP1: ~, Jumper:SolderJumper-3_P1.3mm_Bridged12_Pad1.0x1.5mm, F.Cu at (150.5, 63.5)
- added U6: 74LVC1G175, Package_TO_SOT_SMD:SOT-363_SC-70-6, F.Cu at (150.5, 67.3)
- added U7: 74LVC1GU04, Package_TO_SOT_SMD:SOT-353_SC-70-5, F.Cu at (147.3, 67.7)
- moved C3 13.4 mm to (151.1, 71.1)
- moved D2 1.27 mm to (144.8, 68.6)
Connections:
- C4 pad 1: /~{RESET} -> /~{M2_HALT}
- D3 pad 1: /~{RESET} -> /~{M2_HALT}
- J2 pad 2: /YM_LRCK -> /CLK_8MHz
- J2 pad 6: /YM_SDAT -> /YM_LRCK
- J2 pad 8: GND -> /YM_SDAT
- R2 pad 1: /~{RESET} -> /~{M2_HALT}
- U1 pad 22: VCC -> unconnected-(U1-~{STBY}-Pad22)
- U1 pad 28: Net-(U1-FMOSC) -> /CLK_8MHz
- X1 pad 3: Net-(U1-FMOSC) -> /CLK_8MHz
Routing:
- net /~{M2_HALT}: track 0.00 -> 69.9 mm, vias 0 -> 2
- net /~{RESET}: track 55.9 -> 19.7 mm, vias 0 -> 2
- net GND: track 39.5 -> 61.2 mm, vias 196 -> 192
- net /YM_LRCK: track 13.1 -> 28.7 mm, vias 2 -> 4
- net /CLK_8MHz: track 0.00 -> 14.8 mm
- net VCC: track 82.8 -> 96.2 mm, vias 69 -> 68
- net Net-(U1-FMOSC): track 6.97 -> 0.00 mm
- net Net-(U6-C): track 0.00 -> 4.58 mm, vias 0 -> 2
- net Net-(JP1-A): track 0.00 -> 1.89 mm
- net /YM_SDAT: track 14.5 -> 15.7 mm
- net /AUD_RF: track 75.4 -> 74.2 mm
- net Net-(D2-K): track 3.45 -> 4.57 mm
