File: EPSM YMF288 Modular Famicom Horizontal/EPSM YMF288 Modular Famicom Horizontal.kicad_sch (KiCad schematic)
At the start: 28 parts, among them J1 EPSM_DATA, J2 EPSM_AUDIO, J3 EPSM_SND_OUT, J4 EPSM_ADDR, J5 CONSOLE_M, J6 CARTRIDGE_F, U1 YMF288, U2 74HCT541, U3 74HCT541, U4 74HCT541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

Commit message: Adjust routing
Other:
- title: Expansion Port Sound Module - Modular Famicom H Connector -> EPSM - Modular Famicom H Connector
Changed lines of the file:
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@@
 	(paper "A4")
 	(title_block
-		(title "Expansion Port Sound Module - Modular Famicom H Connector")
+		(title "EPSM - Modular Famicom H Connector")
 		(date "2025-04-17")
 		(rev "r0.1.0")
