File: EPSM YMF288 Modular Famicom Horizontal/EPSM YMF288 Modular Famicom Horizontal.kicad_sch (KiCad schematic)
At the start: 28 parts, among them J1 EPSM_DATA, J2 EPSM_AUDIO, J3 EPSM_SND_OUT, J4 EPSM_ADDR, J5 CONSOLE_M, J6 CARTRIDGE_F, U1 YMF288, U2 74HCT541, U3 74HCT541, U4 74HCT541, U5 74HCT541, X1 SG-8002CA

Commit message: fix: Fix YMF288 wiring and reset
Parts:
- added C11: 0.1uF, Capacitor_SMD:C_0805_2012Metric_Pad1.18x1.45mm_HandSolder, symbol Device:C
- added JP1: (no value), Jumper:SolderJumper-3_P1.3mm_Bridged12_Pad1.0x1.5mm, symbol Jumper:SolderJumper_3_Bridged12
- added U6: 74LVC1G175, Package_TO_SOT_SMD:SOT-363_SC-70-6, symbol 74xGxx:74LVC1G175
- added U7: 74LVC1GU04, Package_TO_SOT_SMD:SOT-353_SC-70-5, symbol 74xGxx:74LVC1GU04DRL
Connections:
- net GND: now also C11.1, U6.2 (GND), U7.3 (GND); no longer J2.8 (Pin_8)
- net VCC: now also C11.2, U6.3 (D), U6.5 (VCC), U7.5 (VCC); no longer U1.22 (VCC)
- net YM_LRCK: now also J2.6 (Pin_6), U7.2; no longer J2.2 (Pin_2)
- net YM_SDAT: now also J2.8 (Pin_8); no longer J2.6 (Pin_6)
- net ~{RESET}: now also JP1.3 (B), U6.4 (Q); no longer C4.1, D3.1 (K), R2.1
- net CLK_8MHz: now reaches U1.28 (MCLK), X1.3 (OUT)
- net CLK_8MHz: now also J2.2 (Pin_2)
- new net: U6.1 (C), U7.4
- new net: JP1.1 (A), U6.6 (~{CLR})
- new net ~{M2_HALT}: C4.1, D3.1 (K), JP1.2 (C), R2.1
- no-connect marks 12 -> 13
Other:
- note added: "<:3 )~"
- note added: "Crystal Oscillator"
- note added: "If not using sync ~{RESET}, unpopulate D flip flop, break jumper and short ~{M2_HALT} to ~{RESET}"
- note added: "Synchronized ~{RESET} signal"
- company: Persune -> Copyright © 2022-2026 Persune
- moved on the sheet: C1, C2, C3, C4, D1, D2, D3, R1, R2, X1
